File: Esquema/TopGame_BitEletronica/TopGame_BitEletronica.kicad_pcb (KiCad board)
At the start: 4 copper layers, 148.5 x 191 mm, 148 parts, among them CN1 Conn_02x12_Counter_Clockwise, J10 8, J11 5, J13 7, J14 2, J15 3, J16 4, J17 +5V, J18 GND, J19 PB/C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

Commit message: Revisão 1 da placa finalizada.
Parts:
- removed ? (x6): , 
- removed REF** (x7): Pad_3mm_furo_1mm, TopGame_BitEletronica:Pad_3mm_furo_1mm
- added J25: GND, TopGame_BitEletronica:Pad_3mm_furo_1mm, F.Cu at (54.3, 152.2)
- added J26: GND, TopGame_BitEletronica:Pad_3mm_furo_1mm, F.Cu at (54.3, 127.3)
- added J27: ~, TopGame_BitEletronica:Pad_3mm_furo_1mm, F.Cu at (40.0, 122.3)
- added J28: ~, TopGame_BitEletronica:Pad_3mm_furo_1mm, F.Cu at (115.7, 172.0)
- added J29: ~, TopGame_BitEletronica:Pad_3mm_furo_1mm, F.Cu at (116.2, 196.5)
- added J30: ~, TopGame_BitEletronica:Pad_3mm_furo_1mm, F.Cu at (112.6, 217.5)
- added J31: ~, TopGame_BitEletronica:Pad_3mm_furo_1mm, F.Cu at (136.7, 219.2)
- added J32: ~, TopGame_BitEletronica:Pad_3mm_furo_1mm, F.Cu at (144.8, 63.8)
- added J33: ~, TopGame_BitEletronica:Pad_3mm_furo_1mm, F.Cu at (156.6, 64.6)
- added J34: ~, TopGame_BitEletronica:Pad_3mm_furo_1mm, F.Cu at (39.7, 148.0)
- J10, J3: value 8 -> 6; footprint TopGame_BitEletronica:Pad_3mm_furo_1mm -> TopGame_BitEletronica:Pin_2mm_Furo_1mm
- J11, J13, J14, J15, J16, J4, J6, J7, J8, J9: footprint TopGame_BitEletronica:Pad_3mm_furo_1mm -> TopGame_BitEletronica:Pin_2mm_Furo_1mm
Connections:
- CI7 pad 10: (no net) -> unconnected-(CI7-Pad10)
- CI7 pad 11: (no net) -> unconnected-(CI7-Pad11)
- CI7 pad 8: (no net) -> unconnected-(CI7-Pad8)
- CI7 pad 9: (no net) -> unconnected-(CI7-Pad9)
Routing:
- net Net-(CI4-PHI2): track 321.5 -> 313.2 mm
- net Net-(CI6-Pin_1): track 71.9 -> 64.3 mm
- net Net-(CI4-LUM2): track 187.9 -> 183.6 mm
- net Net-(CI4-A4): track 392.2 -> 388.1 mm
- net D1: track 488.2 -> 484.7 mm
- net Net-(CI4-D2): track 515.3 -> 512.2 mm
- net Net-(CI4-A5): track 347.7 -> 344.8 mm
- net D0: track 449.2 -> 446.4 mm
- net +5V: track 264.5 -> 261.7 mm
- net Net-(CI4-D5): track 426.8 -> 424.0 mm
- net Net-(CI5-A6): track 251.8 -> 249.1 mm
- net Net-(CI1-Pin_3): track 313.7 -> 310.9 mm
- net Net-(CI4-A0): track 365.5 -> 362.8 mm
- net Net-(CI4-A1): track 345.0 -> 342.3 mm
- net Net-(CI6-Pin_9): track 354.5 -> 351.8 mm
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Other:
- board text added: "CFOLLY Rev 1 08/2024"
- board text added: "Recriado por: Clemar Folly Jr. https://github.com/clemarfolly/BitEletronica-TopGame"
