File: Esquema/TopGame_BitEletronica/TopGame_BitEletronica.kicad_sch (KiCad schematic)
At the start: 161 parts, among them CN1 Conn_02x12_Counter_Clockwise, J1 1, J10 8, J11 5, J12 6, J13 7, J14 2, J15 3, J16 4, J17 +5V, J18 GND, J19 PB/C, J2 1, J20 PAF, J21 SEL., J22 +5V, J23 GND, J24 L4_3, J3 8, J4 5, J5 6, J6 7, J7 2, J8 3, J9 4, SW1 CHAVE CANAL, SW2 CH. LIG/DESL, SW3 PB/C, SW4 DIF ESQ.⊛, SW5 DIF DIR.⊛, SW6 PAF, SW7 SEL., T1 NPN, T2 MPS3563, T3 MPS3906, U1 L7805, Y1 Crystal_Small

Commit message: Revisão 1 da placa finalizada.
Parts:
- added unit 4 of CI7
- added unit 5 of CI7
- added J25, J26: GND, TopGame_BitEletronica:Pad_3mm_furo_1mm, symbol Connector:Conn_01x01_Pin
- added J27, J28, J29, J30, J31, J32, J33, J34: ~, TopGame_BitEletronica:Pad_3mm_furo_1mm, symbol Connector:Conn_01x01_Pin
- J1, J11, J13, J14, J15, J16, J2, J4, J6, J7, J8, J9: footprint TopGame_BitEletronica:Pad_3mm_furo_1mm -> TopGame_BitEletronica:Pin_2mm_Furo_1mm; symbol Connector:Conn_01x01_Male -> Connector:Conn_01x01_Pin
- J10, J3: value 8 -> 6; footprint TopGame_BitEletronica:Pad_3mm_furo_1mm -> TopGame_BitEletronica:Pin_2mm_Furo_1mm; symbol Connector:Conn_01x01_Male -> Connector:Conn_01x01_Pin
- J12: value 6 -> 8; symbol Connector:Conn_01x01_Male -> Connector:Conn_01x01_Pin
- J17, J18, J19, J20, J21, J22, J23, J24: symbol Connector:Conn_01x01_Male -> Connector:Conn_01x01_Pin
- J5: value 6 -> 8; footprint TopGame_BitEletronica:Pad_3mm_furo_1mm -> TopGame_BitEletronica:Pin_2mm_Furo_1mm; symbol Connector:Conn_01x01_Male -> Connector:Conn_01x01_Pin
Connections:
- net +5V: now also J28.1 (Pin_1), J29.1 (Pin_1), J30.1 (Pin_1), J31.1 (Pin_1), J32.1 (Pin_1), J33.1 (Pin_1)
- net GND: now also J25.1 (Pin_1), J26.1 (Pin_1)
- net at C23.1, R20.2, R21.2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: now also J27.1 (Pin_1), J34.1 (Pin_1)
- no-connect marks 29 -> 33
Other:
- company: (none) -> Clemar Folly Jr. - https://www.x.com/clemarfolly
- title: (none) -> Top Game - Bit Eletrônica
- moved on the sheet: C1, C10, C101, C102, C11, C12, C13, C14, C15, C16, C17, C19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
